Commit message: Agregar fisicas, colisiones  plugin de traccion diferencial para gazebo

File: description/robot.urdf.xacro (robot description, xacro)
@@ -2,3 +2,4 @@
 <robot xmlns:xacro="http://www.ros.org/wiki/xacro"  name="robot">
 	<xacro:include filename="robot_core.xacro" />
+	<xacro:include filename="gazebo_control.xacro" />
 </robot>

File: description/robot_core.xacro (robot description, xacro)
@@ -1,4 +1,5 @@
 <?xml version="1.0"?>
 <robot xmlns:xacro="https://www.ros.org/wiki">
+  <!-- colores -->
   <material name="white">
     <color rgba="1 1 1 1"/>
@@ -12,4 +13,5 @@
   <link name="base_link">
   </link>
+  <!-- chasiss -->
   <joint name="chassis_joint" type="fixed">
     <parent link="base_link"/>
@@ -25,5 +27,20 @@
       <material name="white"/>
     </visual>
+    <collision>
+      <origin xyz="0.15 0 0.075"/>
+      <geometry>
+        <box size="0.3 0.3 0.15"/>
+      </geometry>
+    </collision>
+    <inertial>
+      <origin xyz="0.15 0 0.075" rpy="0 0 0"/>
+      <mass value="0.5"/>
+      <inertia ixx="0.0046875" ixy="0.0" ixz="0.0" iyy="0.0046875" iyz="0.0" izz="0.0075"/>
+    </inertial>
   </link>
+  <gazebo reference="chassis">
+    <material>Gazebo/White</material>
+  </gazebo>
+  <!-- left_wheel -->
   <joint name="left_wheel_joint" type="continuous">
     <parent link="base_link"/>
@@ -39,5 +56,19 @@
       <material name="blue"/>
     </visual>
+    <collision>
+      <geometry>
+        <cylinder radius="0.05" length="0.04"/>
+      </geometry>
+    </collision>
+    <inertial>
+      <origin xyz="0 0 0" rpy="0 0 0"/>
+      <mass value="0.1"/>
+      <inertia ixx="0.0000758" ixy="0.0" ixz="0.0" iyy="0.0000758" iyz="0.0" izz="0.000125"/>
+    </inertial>
   </link>
+  <gazebo reference="left_wheel">
+    <material>Gazebo/Blue</material>
+  </gazebo>
+  <!-- right_wheel -->
   <joint name="right_wheel_joint" type="continuous">
     <parent link="base_link"/>
@@ -53,17 +84,46 @@
       <material name="blue"/>
     </visual>
+    <collision>
+      <geometry>
+        <cylinder radius="0.05" length="0.04"/>
+      </geometry>
+    </collision>
+    <inertial>
+      <origin xyz="0 0 0" rpy="0 0 0"/>
+      <mass value="0.1"/>
+      <inertia ixx="0.0000758" ixy="0.0" ixz="0.0" iyy="0.0000758" iyz="0.0" izz="0.000125"/>
+    </inertial>
   </link>
-    <joint name="caster_wheel_joint" type="fixed">
-        <parent link="chassis"/>
-        <child link="caster_wheel"/>
-        <origin xyz="0.24 0 0"/>
-    </joint>
-    <link name="caster_wheel">
-        <visual>
-            <geometry>
-                <sphere radius="0.05"/>
-            </geometry>
-            <material name="black"/>
-        </visual>
-    </link>
+  <gazebo reference="right_wheel">
+    <material>Gazebo/Blue</material>
+  </gazebo>
+  <!-- caster_wheel -->
+  <joint name="caster_wheel_joint" type="fixed">
+      <parent link="chassis"/>
+      <child link="caster_wheel"/>
+      <origin xyz="0.24 0 0"/>
+  </joint>
+  <link name="caster_wheel">
+    <visual>
+      <geometry>
+        <sphere radius="0.05"/>
+       </geometry>
+       <material name="black"/>
+    </visual>
+    <collision>
+      <geometry>
+        <sphere radius="0.05"/>
+      </geometry>
+    </collision>
+    <inertial>
+      <origin xyz="0 0 0" rpy="0 0 0"/>
+      <mass value="0.1"/>
+      <inertia ixx="0.0001" ixy="0.0" ixz="0.0" iyy="0.0001" iyz="0.0" izz="0.0001"/>
+    </inertial>
+  </link>
+  <gazebo reference="caster_wheel">
+    <material>Gazebo/Black</material>
+    <mu1>0.001</mu1>
+    <mu2>0.001</mu2>
+  </gazebo>
 </robot>
